Commit message: saving

File: gazebo_model_files/box.urdf.xacro (robot description, xacro)
@@ -1,5 +1,5 @@
 <?xml version='1.0'?>
 <robot name="experiment_box" xmlns:xacro="http://www.ros.org/wiki/xacro" >
-  <xacro:property name="box_size" value="0.05" />
+  <xacro:property name="box_size" value="0.03" />
   <xacro:property name="box_mass" value="0.05" />
   <pose>0 0 ${box_size/2} 0 0 0</pose>

Commit message: saving

File: gazebo_model_files/box.urdf.xacro (robot description, xacro)
@@ -4,5 +4,5 @@
   <xacro:property name="box_mass" value="0.05" />
   <pose>0 0 ${box_size/2} 0 0 0</pose>
-  <link name="experiemnt_box_link">
+  <link name="experiment_box_link">
     <gravity>true</gravity>
     <inertial>
@@ -37,5 +37,5 @@
     </visual>
   </link>
-  <gazebo reference="experiemnt_box_link">
+  <gazebo reference="experiment_box_link">
     <material>Gazebo/Blue</material>
   </gazebo>
